File: DualDelay.kicad_sch (KiCad schematic)
At the start: 112 parts, among them J1 9V / GND, J2 IN / OUT / GND, SW1 SPDT on-on, U1 PT2399, U2 PT2399, U3 TL072, U4 TL072, U5 TL072, U6 TL072, U7 78L05, U8 78L05

Commit message: v0.2 breadboard: LFO into the TIME 2 / 2k7 node (even depth), 2k7 minimum delay, LM358 LFO; breadboard plan
Co-Authored-By: Claude Opus 5.5 <noreply@anthropic.com>
Parts:
- removed C48: 1u, symbol Device:C
- removed U6: TL072, symbol Amplifier_Operational:TL072
- added C48: 10u, symbol Device:C_Polarized
- added U6: LM358, symbol Amplifier_Operational:LM358
- R19, R28: value 1k -> 2k7
- R40: value 100k -> 33k
Connections:
- net +9V: now also U6.8 (V+)
- net GND: now also U6.4 (V-)
- net SQR: now also U6.7
- net TRI: now also U6.1
- net VB: now also U6.3 (+), U6.6 (-)
- net at R40.2: now also C48.2
- net at R38.2, R39.1: now also U6.5 (+)
- net TMIN_2: now reaches R28.1, RV2.2, RV2.3
- net TMIN_2: now also C48.1
- net at C46.1, R37.2: now also U6.2 (-)
- net TMIN_1: now reaches R19.1, RV1.2, RV1.3
Other:
- note added: "DELAY LINE 1: PT2399 (U1), network as Loop Echo / Small Time. TIME 1 = B50k + 2k7"
- note added: "DELAY LINE 2: PT2399 (U2), network as Loop Echo / Small Time. TIME 2 = B50k + 2k7"
- note added: "~0.5-12 Hz. Injected at the TIME 2 / 2k7 node: the same DEPTH gives the same percentage wobble at any TIME setting."
- note removed: "DELAY LINE 1: PT2399 (U1), network as Loop Echo / Small Time. TIME 1 = 1k + B50k"
- note removed: "DELAY LINE 2: PT2399 (U2), network as Loop Echo / Small Time. TIME 2 = 1k + B50k"
- note removed: "~0.5-12 Hz. Set RATE slow and DEPTH low for a chorus-like spread between the lines."

Commit message: v1.0 SMD board: 1590BB landscape, three jacks on top (OUT DC IN)
- Schematic (A0, ERC 0): footprints + LCSC (all basic except the PT2399s), MLCC,
  one AMS1117-5.0 per PT2399, FB MAX 1 / 2 trims, 3296W RATE / DEPTH trims,
  PJ-646F / A-4118 jacks, status LED, 1x6 SwitchPCB header. v0.2 kept as
  build_dualdelay_v0.2.py.
- Board (Loop Echo geometry, 100 x 83.5 mm): PT2399s and their regulators at
  opposite ends, slotted Taiway SERIES toggle, dual TWIST pot. DRC 0 errors /
  0 unconnected, parity clean, 73 vias.
- Enclosure drilling files (make_enclosure.py); fab files in production/ (gitignored).

Co-Authored-By: Claude Opus 5.5 <noreply@anthropic.com>
Parts:
- removed C1: 100u, symbol Device:C_Polarized
- removed C10, C15, C27: 47u, symbol Device:C_Polarized
- removed C12, C14, C26, C38, C44, C48, C6, C8: 10u, symbol Device:C_Polarized
- removed C47: 4u7, symbol Device:C_Polarized
- removed D1: 1N5817, symbol Device:D_Schottky
- removed D2, D3, D4, D5: 1N4148, symbol Device:D
- removed J1: 9V / GND, symbol Connector_Generic:Conn_01x02
- removed J2: IN / OUT / GND, symbol Connector_Generic:Conn_01x03
- removed RV5: B10k dual, symbol Device:R_Potentiometer_Dual_Separate
- removed RV6: B10k, symbol Device:R_Potentiometer
- removed RV7: 1M, symbol Device:R_Potentiometer_Trim
- removed RV8: 100k, symbol Device:R_Potentiometer_Trim
- removed U7, U8: 78L05, symbol Regulator_Linear:L78L05_TO92
- added C1: 22u, Capacitor_SMD:C_0805_2012Metric_Pad1.18x1.45mm_HandSolder, symbol Device:C
- added C10, C12, C15, C47, C51: 10u, Capacitor_SMD:C_0805_2012Metric_Pad1.18x1.45mm_HandSolder, symbol Device:C
- added C14, C26, C38, C6, C8: 100n, Capacitor_SMD:C_0805_2012Metric_Pad1.18x1.45mm_HandSolder, symbol Device:C
- added C27: 10n, Capacitor_SMD:C_0805_2012Metric_Pad1.18x1.45mm_HandSolder, symbol Device:C
- added C44, C49: 1u, Capacitor_SMD:C_0805_2012Metric_Pad1.18x1.45mm_HandSolder, symbol Device:C
- added C48: 47n, Capacitor_SMD:C_0805_2012Metric_Pad1.18x1.45mm_HandSolder, symbol Device:C
- added C50: 4u7, Capacitor_SMD:C_0805_2012Metric_Pad1.18x1.45mm_HandSolder, symbol Device:C
- added D1: SS14, Diode_SMD:D_SMA, symbol Diode:SS14
- added D2, D3, D4, D5: 1N4148W, Diode_SMD:D_SOD-123, symbol Diode:1N4148W
- added D6: LED, LED_THT:LED_D3.0mm, symbol Device:LED
- added J1: IJ/IN/LED/GND/OUT/OJ, Connector_PinHeader_2.54mm:PinHeader_1x06_P2.54mm_Vertical, symbol Connector_Generic:Conn_01x06
- added J2: INPUT, SuperFreq:Jack_6.35mm_PJ-646F_Horizontal, symbol Connector_Audio:AudioJack3_Switch
- added J3: OUTPUT, SuperFreq:Jack_6.35mm_PJ-646F_Horizontal, symbol Connector_Audio:AudioJack3_Switch
- added J4: DC 9V, SuperFreq:DC_Jack_2.1mm_A-4118_Horizontal, symbol Connector:Barrel_Jack_Switch
- added R41: 4k7, Resistor_SMD:R_0805_2012Metric_Pad1.20x1.40mm_HandSolder, symbol Device:R
- added RV10: 100k, Potentiometer_THT:Potentiometer_Bourns_3296W_Vertical, symbol Device:R_Potentiometer_Trim
- added RV5, RV6: 10k, Potentiometer_THT:Potentiometer_Bourns_3296W_Vertical, symbol Device:R_Potentiometer_Trim
- added RV7: B10k dual, SuperFreq:Potentiometer_9mm_Dual_Vertical_Tayda, symbol Device:R_Potentiometer_Dual_Separate
- added RV8: B10k, Potentiometer_THT:Potentiometer_Alpha_RD901F-40-00D_Single_Vertical, symbol Device:R_Potentiometer
- added RV9: 1M, Potentiometer_THT:Potentiometer_Bourns_3296W_Vertical, symbol Device:R_Potentiometer_Trim
- added U7, U8: AMS1117-5.0, Package_TO_SOT_SMD:SOT-223-3_TabPin2, symbol Regulator_Linear:AMS1117-5.0
- C11, C19, C22, C3, C31, C34, C4, C5: footprint (none) -> Capacitor_SMD:C_0805_2012Metric_Pad1.18x1.45mm_HandSolder; LCSC (none) -> C49678
- C13: value 1n -> 47u; footprint (none) -> Capacitor_SMD:C_1206_3216Metric_Pad1.33x1.80mm_HandSolder; LCSC (none) -> C96123
- C16: value 100n -> 1n; footprint (none) -> Capacitor_SMD:C_0805_2012Metric_Pad1.18x1.45mm_HandSolder; LCSC (none) -> C46653
- C17, C29, C7, C9: value 100n -> 10u; footprint (none) -> Capacitor_SMD:C_0805_2012Metric_Pad1.18x1.45mm_HandSolder; LCSC (none) -> C15850
- C18, C30: value 100n -> 47u; footprint (none) -> Capacitor_SMD:C_1206_3216Metric_Pad1.33x1.80mm_HandSolder; LCSC (none) -> C96123
- C2: value 100n -> 22u; footprint (none) -> Capacitor_SMD:C_0805_2012Metric_Pad1.18x1.45mm_HandSolder; LCSC (none) -> C45783
- C20, C25, C32, C37: value 2n2 -> 100n; footprint (none) -> Capacitor_SMD:C_0805_2012Metric_Pad1.18x1.45mm_HandSolder; LCSC (none) -> C49678
- C21, C33: value 10n -> 100n; footprint (none) -> Capacitor_SMD:C_0805_2012Metric_Pad1.18x1.45mm_HandSolder; LCSC (none) -> C49678
- C23, C28, C35: value 100n -> 2n2; footprint (none) -> Capacitor_SMD:C_0805_2012Metric_Pad1.18x1.45mm_HandSolder; LCSC (none) -> C28260
- C24, C36: footprint (none) -> Capacitor_SMD:C_0805_2012Metric_Pad1.18x1.45mm_HandSolder; LCSC (none) -> C1710
- C39: value 1u -> 10n; footprint (none) -> Capacitor_SMD:C_0805_2012Metric_Pad1.18x1.45mm_HandSolder; LCSC (none) -> C1710
- C40: value 1u -> 2n2; footprint (none) -> Capacitor_SMD:C_0805_2012Metric_Pad1.18x1.45mm_HandSolder; LCSC (none) -> C28260
- C41: value 1u -> 10u; footprint (none) -> Capacitor_SMD:C_0805_2012Metric_Pad1.18x1.45mm_HandSolder; LCSC (none) -> C15850
- C42: footprint (none) -> Capacitor_SMD:C_0805_2012Metric_Pad1.18x1.45mm_HandSolder; LCSC (none) -> C28323
- C43: value 220p -> 1u; footprint (none) -> Capacitor_SMD:C_0805_2012Metric_Pad1.18x1.45mm_HandSolder; LCSC (none) -> C28323
- C45: value 47n -> 1u; footprint (none) -> Capacitor_SMD:C_0805_2012Metric_Pad1.18x1.45mm_HandSolder; LCSC (none) -> C28323
- C46: value 1u -> 220p; footprint (none) -> Capacitor_SMD:C_0805_2012Metric_Pad1.18x1.45mm_HandSolder; LCSC (none) -> C107145
- R1, R11, R13, R14, R15, R16, R17, R2, R20, R22, R23, R24, R25, R26, R33, R34, R35, R38, R6, R7, R8: footprint (none) -> Resistor_SMD:R_0805_2012Metric_Pad1.20x1.40mm_HandSolder; LCSC (none) -> C17414
- R10: footprint (none) -> Resistor_SMD:R_0805_2012Metric_Pad1.20x1.40mm_HandSolder; LCSC (none) -> C149504
- R12, R21: footprint (none) -> Resistor_SMD:R_0805_2012Metric_Pad1.20x1.40mm_HandSolder; LCSC (none) -> C17475
- R18, R27, R29, R31, R36: footprint (none) -> Resistor_SMD:R_0805_2012Metric_Pad1.20x1.40mm_HandSolder; LCSC (none) -> C17513
- R19, R28: footprint (none) -> Resistor_SMD:R_0805_2012Metric_Pad1.20x1.40mm_HandSolder; LCSC (none) -> C17530
- R3, R30, R32, R5: footprint (none) -> Resistor_SMD:R_0805_2012Metric_Pad1.20x1.40mm_HandSolder; LCSC (none) -> C17514
- R37: footprint (none) -> Resistor_SMD:R_0805_2012Metric_Pad1.20x1.40mm_HandSolder; LCSC (none) -> C17713
- R39: footprint (none) -> Resistor_SMD:R_0805_2012Metric_Pad1.20x1.40mm_HandSolder; LCSC (none) -> C17560
- R4, R9: footprint (none) -> Resistor_SMD:R_0805_2012Metric_Pad1.20x1.40mm_HandSolder; LCSC (none) -> C17408
- R40: footprint (none) -> Resistor_SMD:R_0805_2012Metric_Pad1.20x1.40mm_HandSolder; LCSC (none) -> C17633
- RV1, RV2, RV3, RV4: footprint (none) -> Potentiometer_THT:Potentiometer_Alpha_RD901F-40-00D_Single_Vertical; now left out of the parts list
- SW1: footprint (none) -> SuperFreq:SW_Taiway_100_SPDT_PC; now left out of the parts list
- U1, U2: footprint (none) -> Package_SO:SOIC-16_3.9x9.9mm_P1.27mm; LCSC (none) -> C126407
- U3, U4, U5: footprint (none) -> Package_SO:SOIC-8_3.9x4.9mm_P1.27mm; FT Rotation Offset (none) -> 270; LCSC (none) -> C6961
- U6: footprint (none) -> Package_SO:SOIC-8_3.9x4.9mm_P1.27mm; FT Rotation Offset (none) -> 270; LCSC (none) -> C7950
Connections:
- net +9V: now also C9.1, C1.1, C12.1, C6.1, D1.1 (K), R41.1, U7.3 (VI), U8.3 (VI)
- net D2IN: now also C37.1; no longer C34.1
- net DIN_1: now also C24.1; no longer C21.1
- net DIN_2: now also C36.1; no longer C33.1
- net DRY: now also C25.1; no longer C22.1
- net FB1B: now also RV7.1, RV7.6
- net FB2B: now also RV7.3, RV7.4
- net GND: now also C11.2, C13.2, C18.2, C19.2, C20.2, C30.2, C31.2, C32.2, C39.2, C1.2, C10.2, C12.2, C27.2, C48.2, C6.2, C8.2, D2.1 (K), D3.2 (A), D4.1 (K), D5.2 (A), J1.4 (Pin_4), J2.S, J3.S, J4.1, RV10.1, RV8.1, U7.1 (GND), U8.1 (GND); no longer C16.2, C17.2, C21.2, C28.2, C29.2, C33.2, C45.2
- net IN: now also C14.1, J1.2 (Pin_2); no longer C11.1
- net LP1I_1: now also C23.1; no longer C20.1
- net LP1I_2: now also C35.1; no longer C32.1
- net LP1O_1: now also C23.2; no longer C20.2
- net LP1O_2: now also C35.2; no longer C32.2
- net LP2I_1: now also C28.1; no longer C25.1
- net LP2I_2: now also C40.1; no longer C37.1
- net LP2O_1: now also C28.2, C29.1; no longer C25.2
- net LP2O_2: now also C40.2, C41.1; no longer C37.2
- net MIXW: now also C15.1, RV8.2
- net OP1I_1: now also C21.1; no longer C18.1
- net OP1I_2: now also C33.1; no longer C30.1
- net OP1O_1: now also C21.2; no longer C18.2
- net OP1O_2: now also C33.2; no longer C30.2
- net OP2I_1: now also C22.1; no longer C19.1
- net OP2I_2: now also C34.1; no longer C31.1
- net OP2O_1: now also C22.2; no longer C19.2
- net OP2O_2: now also C34.2; no longer C31.2
- net OUT: now also C17.2, J1.5 (Pin_5)
- net RPT_1: now also C26.1, RV7.2; no longer C23.1
- net RPT_2: now also C38.1, RV7.5; no longer C35.1
- net SQR: now also RV9.2, RV9.3
- net TMIN_2: now also C51.1
- net TRI: now also C49.2, C50.1; no longer C46.2
- net V5_1: now also C8.1, U7.2 (VO)
- net V5_2: now also C11.1, C10.1, U8.2 (VO); no longer C9.1
- net VB: now also C13.1
- net W1: now also C44.1, RV5.1; no longer C41.1, RV3.3
- net W2: now also C45.1, RV6.1; no longer C42.1, RV4.3
- net at R22.1: now also C37.2; no longer C34.2
- net at R27.1: now also C41.2
- net at R6.2, R7.2, R8.1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: now also C16.1; no longer C13.1
- net at R8.2, R9.1, U3.7: now also C16.2; no longer C13.2
- net at R40.1: now also RV10.2
- net at R32.1, U4.5 (+): now also C43.2; no longer C40.2
- net at R33.1: now also C44.2; no longer C41.2
- net at R33.2, R34.2, R35.1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: now also C46.1; no longer C43.1
- net at R9.2: now also C17.1
- net at U2.2 (REF): now also C30.1
- net at R40.2: now also C51.2
- net at R31.2: now also C43.1, D4.2 (A), D5.1 (K); no longer C40.1
- net at R29.2: now also C42.1, D2.2 (A), D3.1 (K); no longer C39.1
- net at R36.2: now also C48.1, RV8.3; no longer C45.1
- net at R36.1: now also C47.2
- net at R37.1: now also RV9.1
- net at R35.2, U5.1: now also C46.2, C47.1; no longer C43.2
- net at U2.7 (CC1): now also C31.1; no longer C28.1
- net at R15.2, R16.1, R17.1: now also C27.1; no longer C24.1
- net at R30.1, U4.3 (+): now also C42.2; no longer C39.2
- net at U2.8 (CC0): now also C32.1; no longer C29.1
- net at R37.2, U6.2 (-): now also C49.1; no longer C46.1
- net at R24.2, R25.1, R26.1: now also C39.1; no longer C36.1
- net at R13.1: now also C25.2; no longer C22.2
- net at R7.1: now also C15.2
- net at U1.2 (REF): now also C18.1
- net at R34.1: now also C45.2; no longer C42.2
- net at R14.1: now also C26.2; no longer C23.2
- net at R4.1: now also C14.2; no longer C11.2
- net at U1.7 (CC1): now also C19.1; no longer C16.1
- net at R18.1: now also C29.2
- net at U1.8 (CC0): now also C20.1; no longer C17.1
- net at R23.1: now also C38.2; no longer C35.2
- new net: D1.2 (A), J4.2, J4.3
- new net: D6.2 (A), R41.2
- new net: C50.2, RV10.3
- new net IJ: J1.1 (Pin_1), J2.T
- new net LED_K: D6.1 (K), J1.3 (Pin_3)
- new net OJ: J1.6 (Pin_6), J3.T
- new net WF1: RV3.3, RV5.2, RV5.3
- new net WF2: RV4.3, RV6.2, RV6.3
- no-connect marks 2 -> 10
Other:
- note added: "FB MAX trims: 0 = full feedback (as v0.2); turn up to lower the maximum repeat level."
- note added: "JACKS (board-mounted, top wall), FOOTSWITCH HEADER (SwitchPCB v2), STATUS LED"
- note added: "POWER: DC jack, SS14, VB, AMS1117-5.0 x2"
- note added: "Panel (1590BB landscape): TIME 1, TIME 2, MIX over FB 1, TWIST, FB 2; SERIES toggle; status LED; footswitch. Internal trims: RATE, DEPTH, FB MAX 1 / 2."
- note removed: "POWER: 9 V, VB 4.5 V for the TL072s, one 78L05 per PT2399"
- note removed: "Panel (1590BB): TIME 1, TIME 2, FB 1, FB 2, TWIST, MIX + SERIES toggle. Internal: RATE, DEPTH."
- title: Dual Delay (breadboard) -> Dual Delay

Commit message: Re-route with the 0.4 mm Power net class restored
Power class in DualDelay.kicad_pro (+9V, GND, V5_1, V5_2, VB, D1-A; Default 0.25 mm), board re-routed
(99 vias, DRC 0/0, parity clean; C32 GND pad solid); buildpcb now restores the .kicad_pro at exit.

Co-Authored-By: Claude Opus 5.5 <noreply@anthropic.com>
Other:
- moved on the sheet: C1, C10, C11, C12, C13, C14, C15, C16, C17, C18, C19, C2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
